Commit message: Added room_seeker_description, room_seeker_slam, room_seeker_navigation pakcage. room_seeker_navigation is now developing.

File: ControlLevel2/src_RemotePC/room_seeker_description/urdf/room_seeker.gazebo.xacro (robot description, xacro)
@@ -1,4 +1,4 @@
 <?xml version="1.0"?>
-<robot name="turtlebot3_waffle_pi_sim" xmlns:xacro="http://ros.org/wiki/xacro">
+<robot name="RoomSeeker" xmlns:xacro="http://ros.org/wiki/xacro">
   <xacro:arg name="laser_visual"  default="false"/>
   <xacro:arg name="camera_visual" default="false"/>

File: ControlLevel2/src_RemotePC/room_seeker_description/urdf/room_seeker.urdf.xacro (robot description, xacro)
@@ -1,6 +1,6 @@
 <?xml version="1.0" ?>
-<robot name="room_seeker" xmlns:xacro="http://ros.org/wiki/xacro">
-  <xacro:include filename="$(find room_seeker_remote)/urdf/common_properties.xacro"/>
-  <xacro:include filename="$(find room_seeker_remote)/urdf/room_seeker.gazebo.xacro"/>
+<robot name="RoomSeeker" xmlns:xacro="http://ros.org/wiki/xacro">
+  <xacro:include filename="$(find room_seeker_description)/urdf/common_properties.xacro"/>
+  <xacro:include filename="$(find room_seeker_description)/urdf/room_seeker.gazebo.xacro"/>
   <link name="base_footprint"/>
   <joint name="base_joint" type="fixed">
@@ -14,8 +14,8 @@
       <origin xyz="0.0 0.0 0.0173" rpy="0 0 0"/>
       <geometry>
-        <!-- <mesh filename="package://room_seeker_remote/meshes/bases/waffle_pi_base.stl" scale="0.001 0.001 0.001"/> -->
-        <mesh filename="package://room_seeker_remote/meshes/bases/MecanumCarBase.stl" scale="0.0001 0.0001 0.0001"/>
-      </geometry>
-      <material name="light_black"/>
+        <!-- <mesh filename="package://room_seeker_description/meshes/bases/waffle_pi_base.stl" scale="0.001 0.001 0.001"/> -->
+        <mesh filename="package://room_seeker_description/meshes/bases/MecanumCarBase.stl" scale="0.0001 0.0001 0.0001"/>
+      </geometry>
+      <material name="brown"/>
     </visual>
     <collision>
@@ -45,5 +45,5 @@
       <origin xyz="0 0 0" rpy="0 0 0"/>
       <geometry>
-        <mesh filename="package://room_seeker_remote/meshes/wheels/RightMecanumWheel.stl" scale="0.00001 0.00001 0.00001"/>
+        <mesh filename="package://room_seeker_description/meshes/wheels/RightMecanumWheel.stl" scale="0.00001 0.00001 0.00001"/>
       </geometry>
       <material name="dark"/>
@@ -74,5 +74,5 @@
       <origin xyz="0 0 0" rpy="0 0 0"/>
       <geometry>
-        <mesh filename="package://room_seeker_remote/meshes/wheels/LeftMecanumWheel.stl" scale="0.0001 0.0001 0.0001"/>
+        <mesh filename="package://room_seeker_description/meshes/wheels/LeftMecanumWheel.stl" scale="0.0001 0.0001 0.0001"/>
       </geometry>
       <material name="dark"/>
@@ -103,5 +103,5 @@
       <origin xyz="0 0 0" rpy="0 0 0"/>
       <geometry>
-        <mesh filename="package://room_seeker_remote/meshes/wheels/RightMecanumWheel.stl" scale="0.00001 0.00001 0.00001"/>
+        <mesh filename="package://room_seeker_description/meshes/wheels/RightMecanumWheel.stl" scale="0.00001 0.00001 0.00001"/>
       </geometry>
       <material name="dark"/>
@@ -132,5 +132,5 @@
       <origin xyz="0 0 0" rpy="0 0 0"/>
       <geometry>
-        <mesh filename="package://room_seeker_remote/meshes/wheels/LeftMecanumWheel.stl" scale="0.0001 0.0001 0.0001"/>
+        <mesh filename="package://room_seeker_description/meshes/wheels/LeftMecanumWheel.stl" scale="0.0001 0.0001 0.0001"/>
       </geometry>
       <material name="dark"/>
@@ -166,5 +166,5 @@
       <origin xyz="0 0 0.0" rpy="0 0 0"/>
       <geometry>
-        <mesh filename="package://room_seeker_remote/meshes/sensors/lds.stl" scale="0.001 0.001 0.001"/>
+        <mesh filename="package://room_seeker_description/meshes/sensors/lds.stl" scale="0.001 0.001 0.001"/>
       </geometry>
       <material name="dark"/>
