Commit message: Bug fixes. Added hardware schematics of MotorNode & SensorNode

File: Level2_Remote/room_seeker_description/urdf/room_seeker.urdf.xacro (robot description, xacro)
@@ -157,14 +157,15 @@
   </joint>
   <link name="imu_link"/>
+  <!-- Lidar part -->
   <joint name="scan_joint" type="fixed">
     <parent link="base_link"/>
     <child link="base_scan"/>
-    <origin xyz="-0.064 0 0.122" rpy="0 0 0"/>
+    <origin xyz="-0.132 0.0 0.0883" rpy="0 0 0"/>
   </joint>
   <link name="base_scan">
     <visual>
-      <origin xyz="0 0 0.0" rpy="0 0 0"/>
-      <geometry>
-        <mesh filename="package://room_seeker_description/meshes/sensors/lds.stl" scale="0.001 0.001 0.001"/>
+      <origin xyz="0.0 0.0 0.0" rpy="0 0 0"/>
+      <geometry>
+        <mesh filename="package://room_seeker_description/meshes/sensors/RP-lidar-A1.stl" scale="0.001 0.001 0.001"/>
       </geometry>
       <material name="dark"/>
